File: pcb/maskrom-adapter/maskrom-adapter.kicad_pcb (KiCad board)
At the start: 2 copper layers, 15 x 30 mm, 2 parts, among them IC1 Maskrom, IC2 M29F160FB5AN6F2

Commit message: Maskrom adapter V1
Parts:
- added R1: 1K, LED_SMD:LED_0805_2012Metric_Pad1.15x1.40mm_HandSolder, F.Cu at (149.7, 106.5)
Connections:
- IC2 pad 11: /VCC -> Net-(IC2-BYTE#)
- IC2 pad 12: /VCC -> Net-(IC2-BYTE#)
- IC2 pad 47: /BYTE -> Net-(IC2-BYTE#)
Routing:
- net Net-(IC2-BYTE#): track 0.00 -> 31.5 mm, vias 0 -> 3
- net /A0: track 0.00 -> 11.5 mm
- net /A16: track 0.00 -> 11.5 mm
- net /CE: track 0.00 -> 10.9 mm, vias 0 -> 1
- net /OE: track 0.00 -> 9.56 mm, vias 0 -> 1
- net /D15: track 0.00 -> 9.50 mm, vias 0 -> 1
- net /VCC: track 0.00 -> 9.13 mm
- net /D11: track 0.00 -> 9.12 mm
- net /A15: track 0.00 -> 9.05 mm
- net /A1: track 0.00 -> 8.99 mm
- net /D0: track 0.00 -> 8.96 mm, vias 0 -> 1
- net /D7: track 0.00 -> 8.87 mm, vias 0 -> 1
- net /A14: track 0.00 -> 8.73 mm, vias 0 -> 1
- net /A2: track 0.00 -> 8.24 mm, vias 0 -> 1
- net /D8: track 0.00 -> 8.19 mm, vias 0 -> 1
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- added copper zone on B.Cu, net /GND
- added copper zone on F.Cu, net /GND
Other:
- board text added: "1"
- board text added: "22"
- board text added: "44"
