File: pcb/maskrom-adapter/maskrom-adapter.kicad_sch (KiCad schematic)
At the start: 2 parts, among them IC1 Maskrom, IC2 M29F160FB5AN6F2

Commit message: Maskrom adapter V1
Parts:
- added R1: 1K, LED_SMD:LED_0805_2012Metric_Pad1.15x1.40mm_HandSolder, symbol Device:R_Small
Connections:
- net BYTE: no longer IC2.47 (BYTE#)
- net VCC: now also R1.1; no longer IC2.11 (WE#), IC2.12 (RP#)
- new net: IC2.11 (WE#), IC2.12 (RP#), IC2.47 (BYTE#), R1.2
Other:
- title: Reverse Engineered XK-403 -> XK-403 Maskrom TSOP48 Adapter
Changed lines of the file:
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@@
 	(paper "A4")
 	(title_block
-		(title "Reverse Engineered XK-403")
-		(date "2023-03-08")
+		(title "XK-403 Maskrom TSOP48 Adapter")
+		(date "2025-04-26")
+	)
+	(junction
+		(at 100.33 73.66)
+		(diameter 0)
+		(color 0 0 0 0)
 	)
 	(no_connect
@@
 	(wire
 		(pts
-			(xy 96.52 76.2) (xy 105.41 76.2)
+			(xy 99.06 73.66) (xy 100.33 73.66)
 		)
 		(stroke
@@
 	(wire
 		(pts
-			(xy 96.52 73.66) (xy 105.41 73.66)
+			(xy 100.33 73.66) (xy 105.41 73.66)
 		)
 		(stroke
@@
 		)
 	)
+	(wire
+		(pts
+			(xy 100.33 76.2) (xy 100.33 73.66)
+		)
+		(stroke
+			(width 0)
+			(type default)
+		)
+	)
+	(wire
+		(pts
+			(xy 87.63 73.66) (xy 93.98 73.66)
+		)
+		(stroke
+			(width 0)
+			(type default)
+		)
+	)
+	(wire
+		(pts
+			(xy 105.41 76.2) (xy 100.33 76.2)
+		)
+		(stroke
+			(width 0)
+			(type default)
+		)
+	)
+	(wire
+		(pts
+			(xy 148.59 39.37) (xy 100.33 39.37)
+		)
+		(stroke
+			(width 0)
+			(type default)
+		)
+	)
+	(wire
+		(pts
+			(xy 100.33 39.37) (xy 100.33 73.66)
+		)
+		(stroke
+			(width 0)
+			(type default)
+		)
+	)
+	(wire
+		(pts
+			(xy 148.59 50.8) (xy 148.59 39.37)
+		)
+		(stroke
+			(width 0)
+			(type default)
+		)
+	)
+	(wire
+		(pts
+			(xy 138.43 50.8) (xy 148.59 50.8)
+		)
+		(stroke
+			(width 0)
+			(type default)
+		)
+	)
 	(label "D7"
 		(at 198.12 86.36 0)
@@
 		)
 	)
-	(label "VCC"
-		(at 96.52 76.2 0)
-		(effects
-			(font
-				(size 1.27 1.27)
-			)
-			(justify left bottom)
-		)
-	)
 	(label "A2"
 		(at 105.41 104.14 180)
@@
 		)
 	)
-	(label "BYTE"
-		(at 138.43 50.8 0)
-		(effects
-			(font
-				(size 1.27 1.27)
-			)
-			(justify left bottom)
-		)
-	)
 	(label "D6"
 		(at 198.12 91.44 0)
@@
 	)
 	(label "VCC"
-		(at 96.52 73.66 0)
+		(at 87.63 73.66 0)
 		(effects
 			(font
@@
 		)
 	)
+	(symbol
+		(lib_id "Device:R_Small")
+		(at 96.52 73.66 90)
+		(unit 1)
+		(exclude_from_sim no)
+		(in_bom yes)
+		(on_board yes)
+		(dnp no)
+		(fields_autoplaced yes)
+		(property "Reference" "R1"
+			(at 96.52 68.58 90)
+			(effects
+				(font
+					(size 1.016 1.016)
+				)
+			)
+		)
+		(property "Value" "1K"
+			(at 96.52 71.12 90)
+			(effects
+				(font
+					(size 1.27 1.27)
+				)
+			)
+		)
+		(property "Footprint" "LED_SMD:LED_0805_2012Metric_Pad1.15x1.40mm_HandSolder"
+			(at 96.52 73.66 0)
+			(effects
+				(font
+					(size 1.27 1.27)
+				)
+				(hide yes)
+			)
+		)
+		(property "Datasheet" "~"
+			(at 96.52 73.66 0)
+			(effects
+				(font
+					(size 1.27 1.27)
+				)
+				(hide yes)
+			)
+		)
+		(property "Description" "Resistor, small symbol"
+			(at 96.52 73.66 0)
+			(effects
+				(font
+					(size 1.27 1.27)
+				)
+				(hide yes)
+			)
+		)
+		(pin "2"
+		)
+		(pin "1"
+		)
+		(instances
+			(project ""
+				(path "/5081f4fb-0c92-4cfc-8c52-39777c6d96ed"
+					(reference "R1")
+					(unit 1)
+				)
+			)
+		)
+	)
