File: pcb/flash-32mbit/flash-32mbit.kicad_pcb (KiCad board)
At the start: 2 copper layers, 96.3 x 76.2 mm, 33 parts, among them U1 LH28F320SKTD-L70, U2 AS6C1008-55SIN, U3 SN74LVC1G04, U4 RP2040-Tiny, U5 MCP23S17T-E/SS, U6 MCP23S17T-E/SS, U7 MCP23S17T-E/SS

Commit message: Marking SRAM pullup R14 do not populate
Parts:
- R1: value 1K2 -> 1K
Other:
- board text removed: "JLCJLCJLCJLC"
