File: pcb/flash-32mbit/flash-32mbit.kicad_sch (KiCad schematic)
At the start: 32 parts, among them U1 LH28F320SKTD-L70, U2 AS6C1008-55SIN, U3 SN74LVC1G04, U4 RP2040-Tiny, U5 MCP23S17T-E/SS, U6 MCP23S17T-E/SS, U7 MCP23S17T-E/SS

Commit message: Marking SRAM pullup R14 do not populate
Parts:
- R1: value 1K2 -> 1K
- R14: now not fitted; now left out of the parts list
Changed lines of the file:
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@@
 		(unit 1)
 		(exclude_from_sim no)
-		(in_bom yes)
+		(in_bom no)
 		(on_board yes)
-		(dnp no)
+		(dnp yes)
 		(fields_autoplaced yes)
 		(property "Reference" "R14"
@@
 			)
 		)
-		(property "Value" "1K2"
+		(property "Value" "1K"
 			(at 100.33 251.46 90)
 			(effects
